File: hardware/rpi-cm4-board/rpi-cm4-board.kicad_pcb (KiCad board)
At the start: 4 copper layers, 85.5 x 82 mm, 66 parts, among them J1 Micro_SD_Card_Det, J2 Screw_Terminal_01x02, J3 Screw_Terminal_01x02, J4 Screw_Terminal_01x02, J5 RJ45_Amphenol_RJMG1BD3B8K1ANR, U10 ISOW7741, U11 THVD1450DR, U3 74LVC1G07SE-7, U5 1-215297-5, U6 RT9742GGJ5, U7 R1500H050B-T1-FE, U8 ISOW7741, U9 THVD1450DR

Commit message: design rules comliance review 1
Parts:
- removed the ? at (175.0, 130.0)
- removed the ? at (97.5, 130.0)
- removed the ? at (97.5, 56.0)
- added ?: , , F.Cu at (117.2, 56.8)
- added ?: , , F.Cu at (175.0, 130.2)
- added ?: , , F.Cu at (97.4, 130.2)
- added ?: , , F.Cu at (150.3, 56.8)
- added ?: , , F.Cu at (117.5, 104.8)
- added ?: , , F.Cu at (150.5, 104.8)
- added ?: , , F.Cu at (97.4, 55.8)
- moved TP1 8.64 mm to (108.0, 54.8)
- moved J3 0.95 mm to (151.2, 130.5)
- moved J4 0.78 mm to (163.0, 130.5)
Routing:
- net /CM4 GPIO/RXD0: track 56.1 -> 67.3 mm
- net GND: track 138.5 -> 147.9 mm, vias 44 -> 40
- net Net-(D1-K): track 14.0 -> 5.46 mm
- net /CM4 GPIO/TXD3: track 33.5 -> 40.4 mm
- net +5V: track 114.8 -> 121.1 mm
- net /CM4 GPIO/DE3: track 25.5 -> 29.2 mm
- net /CM4 GPIO/TXD0: track 56.8 -> 60.3 mm
- net /CM4 GPIO/CTS0: track 55.8 -> 59.1 mm
- net /RX485/RS485_RXD3: track 36.7 -> 33.8 mm
- net Net-(Module1A-PI_nLED_Activity): track 51.6 -> 53.7 mm
- net /CM4 GPIO/GPIO_VREF: track 24.1 -> 26.1 mm
- net /CM4 GPIO/ETH_LEDY: track 64.0 -> 62.7 mm
- net /CM4 GPIO/ETH_LEDG: track 48.2 -> 47.0 mm
- net /RX485/RS485_DE3: track 37.7 -> 36.6 mm
- net +3.3V: track 98.6 -> 99.4 mm
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
Commit message: I need a cyberdeck
Parts:
- added C15: 1000p, Capacitor_SMD:C_0603_1608Metric, F.Cu at (77.8, 150.0)
- added C16: 4u7, Capacitor_SMD:CP_Elec_5x3, F.Cu at (97.4, 161.5)
- added C17: 10u, Capacitor_SMD:C_0603_1608Metric, F.Cu at (77.8, 152.5)
- added C18: 1u, Capacitor_SMD:C_0603_1608Metric, F.Cu at (77.8, 155.0)
- added C19: 10u, Capacitor_SMD:C_0603_1608Metric, F.Cu at (77.8, 157.5)
- added D2: 1N5819WS, Diode_SMD:D_SOD-323, F.Cu at (95.1, 166.4)
- added D3: LED, LED_SMD:LED_0603_1608Metric, F.Cu at (99.3, 166.2)
- added D4: 1N5819WS, Diode_SMD:D_SOD-323, F.Cu at (95.1, 169.3)
- added J5: USB_C_Receptacle_PowerOnly_6P, Connector_USB:USB_C_Receptacle_GCT_USB4125-xx-x-0190_6P_TopMnt_Horizontal, F.Cu at (93.7, 153.6)
- added J6: Conn_01x02_Socket, Connector_JST:JST_EH_S2B-EH_1x02_P2.50mm_Horizontal, F.Cu at (79.3, 169.0)
- added Q1: AO3401A, Package_TO_SOT_SMD:SOT-23, F.Cu at (90.2, 169.5)
- added R15: 1M, Resistor_SMD:R_0603_1608Metric, F.Cu at (77.8, 160.0)
- added R16: 5k1, Resistor_SMD:R_0603_1608Metric, F.Cu at (81.8, 150.0)
- added R17: 5k1, Resistor_SMD:R_0603_1608Metric, F.Cu at (81.8, 152.5)
- added R18: 10K, Resistor_SMD:R_0603_1608Metric, F.Cu at (81.8, 155.0)
- added R19: 10K, Resistor_SMD:R_0603_1608Metric, F.Cu at (81.8, 157.5)
- added R20: 10K, Resistor_SMD:R_0603_1608Metric, F.Cu at (81.8, 160.0)
- added R21: 10K, Resistor_SMD:R_0603_1608Metric, F.Cu at (85.8, 150.0)
- added R22: 10K, Resistor_SMD:R_0603_1608Metric, F.Cu at (85.8, 152.5)
- added R23: 10K, Resistor_SMD:R_0603_1608Metric, F.Cu at (85.8, 155.0)
- added U7: MCP73831-2-OT, Package_TO_SOT_SMD:SOT-23-5, F.Cu at (90.4, 160.4)
- added U8: XC6220B331MR, Package_TO_SOT_SMD:SOT-23-5, F.Cu at (90.4, 165.1)
- renumbered C5 to C10, C12 to C11, C6 to C12, C7 to C14, C14 to C3, C8 to C4, C15 to C5, C9 to C6, C16 to C7, C10 to C8, C11 to C9, FB3 to FB1, FB4 to FB2, FB1 to FB3, FB2 to FB4, J5 to J1, J1 to J2, J4 to J3, J3 to J4, R3 to R1, R11 to R10, R14 to R11, R15 to R12, R12 to R13, R13 to R14, R1 to R2, R2 to R3, R9 to R6, R10 to R7, R7 to R8, R8 to R9, TP2 to TP1, TP3 to TP2, TP4 to TP3, TP1 to TP4, TP7 to TP5, TP8 to TP6, TP9 to TP7, U5 to U1, U6 to U2, U10 to U3, U8 to U4, U11 to U5, U9 to U6
